File: RPi_Zero_pHat_Template.kicad_pcb (KiCad board)
At the start: 2 copper layers, 65 x 30.5 mm, 6 parts, among them J1 RPi_GPIO, J2 RPi_GPIO

Commit message: Version 1.0 complete
Parts:
- removed the J1 at (45.0, 28.0)
- added J2: Screw_Terminal_01x03, TerminalBlock:TerminalBlock_bornier-3_P5.08mm, F.Cu at (19.6, 44.6)
- added J3: Screw_Terminal_01x03, TerminalBlock:TerminalBlock_bornier-3_P5.08mm, F.Cu at (41.0, 47.0)
- added J4: Screw_Terminal_01x03, TerminalBlock:TerminalBlock_bornier-3_P5.08mm, F.Cu at (59.6, 47.0)
- added J5: Screw_Terminal_01x03, TerminalBlock:TerminalBlock_bornier-3_P5.08mm, F.Cu at (70.5, 34.5)
- added R1: 4.7K, Resistor_THT:R_Axial_DIN0207_L6.3mm_D2.5mm_P10.16mm_Horizontal, F.Cu at (49.1, 36.4)
- renumbered J2 to J1
Connections:
- J1 pad 1: Net-(J2-Pad1) -> /V+
- J1 pad 25: Net-(J2-Pad25) -> /GND
- J1 pad 7: Net-(J2-Pad7) -> /IO
Routing:
- net /IO: track 0.00 -> 77.1 mm
- added copper zone on B.Cu, net /GND
- added copper zone on F.Cu, net /V+
Other:
- board size 65 x 30.5 mm -> 65 x 30 mm
- board text added: "+"
- board text added: "4.7K"
- board text added: "By @grajohnt"
- board text added: "GND"
- board text added: "IO"
- board text added: "OneWire uHat"
- board text added: "This side towards the pi, please"
- board text removed: "Select one of these board edges depending upon the type of socket that is used."
